File: PCB/DCD.kicad_pcb (KiCad board)
At the start: 2 copper layers, 80 x 125 mm, 64 parts, among them J1 USB_C_Receptacle_USB2.0_16P, J10 Conn_01x06, J3 Conn_01x04, J4 Conn_01x08, J5 Conn_01x06, J6 AudioJack3, J7 AudioJack3, J9 Conn_01x03, Q1 AO3401A, Q2 2N7002, Q3 AO3401A, Q4 AO3401A, Q5 2N7002, SW1 RESET, SW2 SW_SPDT, SW3 BOOT, SW4 FF, SW5 RotaryEncoder_Switch, SW6 BACK, SW7 PLAY, SW8 SETUP, U1 ESP32-S3-WROOM-1, U2 USBLC6-2SC6, U3 TPA6132A2RTE, U4 AP2112K-3.3, U5 MCP73831-2-OT

Commit message: Add files via upload
Connections:
- J4 pad 2: /SPI_MOSI -> /SPI_SCK
- J4 pad 3: /SPI_SCK -> /SPI_MOSI
Routing:
- net /SPI_SCK: track 108.3 -> 140.2 mm, vias 1 -> 8
- net /SPI_MOSI: track 118.6 -> 118.0 mm, vias 2 -> 4
