File: PCB/DCD.kicad_sch (KiCad schematic)
At the start: 82 parts, among them J1 USB_C_Receptacle_USB2.0_16P, J10 Conn_01x06, J3 Conn_01x04, J4 Conn_01x08, J5 Conn_01x06, J6 AudioJack3, J7 AudioJack3, J9 Conn_01x03, Q1 AO3401A, Q2 2N7002, Q3 AO3401A, Q4 AO3401A, Q5 2N7002, SW1 RESET, SW2 SW_SPDT, SW3 BOOT, SW4 FF, SW5 RotaryEncoder_Switch, SW6 BACK, SW7 PLAY, SW8 SETUP, U1 ESP32-S3-WROOM-1, U2 USBLC6-2SC6, U3 TPA6132A2RTE, U4 AP2112K-3.3, U5 MCP73831-2-OT

Commit message: Add files via upload
Connections:
- net SPI_MOSI: now also J4.3 (Pin_3); no longer J4.2 (Pin_2)
- net SPI_SCK: now also J4.2 (Pin_2); no longer J4.3 (Pin_3)
Changed lines of the file:
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@@
 		)
 	)
-	(label "SPI_SCK"
+	(label "SPI_MOSI"
 		(at 237.49 176.53 0)
 		(effects
@@
 		)
 	)
-	(label "SPI_MOSI"
+	(label "SPI_SCK"
 		(at 237.49 173.99 0)
 		(effects
